File: Impedance_Analyzer_V2_KiCAD/Impedance_Analyzer_V2.kicad_sch (KiCad schematic)
At the start: 32 parts, among them J1 Conn_Coaxial, J11 Screw_Terminal_01x03, J2 Conn_Coaxial, J3 Conn_Coaxial, J4 Conn_Coaxial, J5 Conn_Coaxial, J6 Conn_Coaxial, J7 Conn_Coaxial, U1 LM358, U2 LM358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

Commit message: Gerbers
Parts:
- added C15: 1n, Capacitor_SMD:C_0805_2012Metric, symbol Device:C
- added C16, C25: 10n, Capacitor_SMD:C_0805_2012Metric, symbol Device:C
- added J10, J12, J13, J14, J15, J16: Conn_02x02_Counter_Clockwise, Connector_PinHeader_2.54mm:PinHeader_2x02_P2.54mm_Vertical, symbol Connector_Generic:Conn_02x02_Counter_Clockwise
- added R11, R12, R22: 1k, Resistor_SMD:R_1206_3216Metric, symbol Device:R
- added R14, R16: 10k, Resistor_SMD:R_1206_3216Metric, symbol Device:R
- added R15, R17: 50, Resistor_SMD:R_1206_3216Metric, symbol Device:R
- R2: value 0 -> 10k
Connections:
- net GND: now also R2.2, C15.2, C16.2, C25.2, R16.2
- net IMon+: now also R14.2
- net IMon-: now also J13.1 (Pin_1), J13.2 (Pin_2); no longer BUF2.6 (Out), R18.1
- net at R8.1, U4.1 (Rg): now also R12.1
- net at U4.8 (Rg): now also J12.3 (Pin_3), J12.4 (Pin_4); no longer R8.2
- net at J1.1 (In): now also R22.2; no longer U1.3 (+)
- net at R2.1, U1.7: now also R15.1; no longer BUF1.3 (In)
- net at R10.2, R3.1, U1.6 (-): no longer R2.2
- net at R1.1, U1.5 (+): now also J16.1 (Pin_1), J16.2 (Pin_2); no longer C1.1
- net at R7.2, U3.1 (Rg): now also R11.1
- net at U3.8 (Rg): now also J10.3 (Pin_3), J10.4 (Pin_4); no longer R7.1
- net at U2.1: now also R16.1, R17.1; no longer BUF2.3 (In)
- new net: J15.1 (Pin_1), J15.2 (Pin_2), R22.1, U1.3 (+)
- new net: C1.1, J16.4 (Pin_4)
- new net: J10.2 (Pin_2), R7.1
- new net: J12.2 (Pin_2), R8.2
- new net: J13.3 (Pin_3), J14.2 (Pin_2), R18.1
- new net: BUF2.3 (In), R17.2
- new net: BUF2.6 (Out), J14.3 (Pin_3), J14.4 (Pin_4)
- new net: BUF1.3 (In), R15.2
- new net: J12.1 (Pin_1), R12.2
- new net: C16.1, J15.3 (Pin_3)
- new net: C15.1, J15.4 (Pin_4)
- new net: J13.4 (Pin_4), J14.1 (Pin_1), R14.1
- new net: J10.1 (Pin_1), R11.2
- new net: C25.1, J16.3 (Pin_3)
Other:
- note added: "Should be similar to shunt (R18 or 14) Does not need to be precision"
- note removed: "Should be similar to R18 Does not need to be precision"
- moved on the sheet: BUF1, BUF2, C1, C3, J1, J4, J5, R1, R10, R2, R21, R3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
