File: Impedance_Analyzer_V2_KiCAD/CurveTracer.kicad_sch (KiCad schematic)
At the start: 11 parts, among them J19 Conn_02x02_Counter_Clockwise, J20 Conn_Coaxial, J21 Conn_02x02_Counter_Clockwise, U1 AD8022, U7 INA129

Commit message: Update Impedance board
Parts:
- J20: footprint Connector_Coaxial:BNC_TEConnectivity_1478204_Vertical -> Eli_Lib:31-5486-1010 BNC Panel RA
Changed lines of the file:
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@@
       (effects (font (size 1.27 1.27)) (justify left))
     )
-    (property "Footprint" "Connector_Coaxial:BNC_TEConnectivity_1478204_Vertical" (id 2) (at 152.4 67.31 0)
+    (property "Footprint" "Eli_Lib:31-5486-1010 BNC Panel RA" (id 2) (at 152.4 67.31 0)
       (effects (font (size 1.27 1.27)) hide)
     )
