File: Impedance_Analyzer_V3_KiCAD/Impedance_Analyzer_V3/Impedance_Analyzer_V3.kicad_pcb (KiCad board)
At the start: 2 copper layers, 94.4 x 90 mm, 87 parts, among them J1 Conn_Coaxial, J10 Conn_02x02_Counter_Clockwise, J11 Screw_Terminal_01x03, J12 Conn_02x02_Counter_Clockwise, J13 Conn_02x02_Counter_Clockwise, J14 Conn_02x02_Counter_Clockwise, J15 Conn_02x02_Counter_Clockwise, J16 Conn_02x02_Counter_Clockwise, J17 Conn_02x02_Counter_Clockwise, J2 Conn_Coaxial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

Commit message: V2Rev B update schematic and add V3 folder
Parts:
- added C26: 100n, Capacitor_SMD:C_0805_2012Metric, F.Cu at (133.2, 117.2)
- added C27: 100n, Capacitor_SMD:C_0805_2012Metric, F.Cu at (132.0, 115.2)
- added R25: 1k, Resistor_SMD:R_1206_3216Metric, B.Cu at (126.7, 112.8)
- added R26: 100, Resistor_SMD:R_1206_3216Metric, B.Cu at (126.8, 110.5)
- added U6: MUX509ID, Package_SO:SOIC-16_3.9x9.9mm_P1.27mm, B.Cu at (133.2, 113.2)
- C11, C12, C13, C2: footprint Capacitor_SMD:C_1206_3216Metric_Pad1.33x1.80mm_HandSolder -> Capacitor_Tantalum_SMD:CP_EIA-6032-20_AVX-F_Pad2.25x2.35mm_HandSolder
- C4, C6: footprint Capacitor_THT:CP_Radial_D5.0mm_P2.00mm -> Capacitor_THT:CP_Radial_D5.0mm_P2.50mm
- J17: value Conn_02x02_Counter_Clockwise -> Screw_Terminal_01x03; footprint Connector_PinHeader_2.54mm:PinHeader_2x02_P2.54mm_Vertical -> TerminalBlock:TerminalBlock_bornier-3_P5.08mm
- R23: value DNP -> 100k; moved to B.Cu
- R24: moved to B.Cu
- moved R24 42.7 mm to (126.8, 115.0)
- moved R23 38.9 mm to (126.8, 117.2), turned to 180 degrees
- moved J17 29.3 mm to (119.2, 57.0), turned to 0 degrees
- moved R9 6.04 mm to (142.5, 73.5)
Connections:
- net InputSig renamed Net-(J1-Pad1)
- net Net-(BUF2-Pad6) renamed Buf2Out
- J17 pad 1: Net-(R9-Pad1) -> GND
- J17 pad 3: IOut -> Net-(J17-Pad3)
- R23 pad 1: Net-(R15-Pad1) -> Net-(R23-Pad1)
- R23 pad 2: Net-(BUF1-Pad6) -> IMon+
- R24 pad 1: Net-(J17-Pad2) -> Net-(R24-Pad1)
- R24 pad 2: Net-(BUF1-Pad6) -> IMon+
- R9 pad 1: Net-(R9-Pad1) -> IOut
Routing:
- net Net-(J17-Pad2): track 3.05 -> 77.0 mm
- net Net-(J17-Pad3): track 0.00 -> 73.0 mm
- net IMon+: track 47.5 -> 62.2 mm, vias 0 -> 1
- net +5VP: track 241.6 -> 254.4 mm, vias 10 -> 13
- net Net-(R25-Pad1): track 0.00 -> 11.3 mm
- net Net-(R26-Pad1): track 0.00 -> 10.6 mm
- net Net-(R23-Pad1): track 0.00 -> 9.89 mm
- net Net-(R24-Pad1): track 0.00 -> 8.62 mm
- net Buf2Out: track 11.3 -> 18.8 mm
- net -5V: track 225.0 -> 232.4 mm, vias 15 -> 16
- net Net-(BUF1-Pad6): track 39.1 -> 33.1 mm
- net Net-(R15-Pad1): track 37.5 -> 31.7 mm
- net GND: track 10.2 -> 15.6 mm, vias 200 -> 226
- net IOut: track 14.9 -> 10.2 mm
- net IMon-: track 5.16 -> 9.45 mm
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Other:
- board text added: "Impedance Analyzer V2 Rev A Eli Mattingly 29 DEC 2021"
- board text removed: "I-Mon Gain Select"
- board text removed: "Impedance Analyzer V2 Rev B Eli Mattingly 31 JUL 2022"
- board text removed: "Input LP Filter"
- board text removed: "J17 Pick R to match R-Shunt value"
- board text removed: "TVS"
- board text removed: "V-Mon Gain Select"
