File: Impedance_Analyzer_V3_KiCAD/Impedance_Analyzer_V3/Impedance_Analyzer_V3.kicad_sch (KiCad schematic)
At the start: 51 parts, among them J1 Conn_Coaxial, J10 Conn_02x02_Counter_Clockwise, J11 Screw_Terminal_01x03, J12 Conn_02x02_Counter_Clockwise, J13 Conn_02x02_Counter_Clockwise, J14 Conn_02x02_Counter_Clockwise, J15 Conn_02x02_Counter_Clockwise, J16 Conn_02x02_Counter_Clockwise, J17 Conn_02x02_Counter_Clockwise, J2 Conn_Coaxial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

Commit message: V2Rev B update schematic and add V3 folder
Parts:
- removed J17: Conn_02x02_Counter_Clockwise, Connector_PinHeader_2.54mm:PinHeader_2x02_P2.54mm_Vertical, symbol Connector_Generic:Conn_02x02_Counter_Clockwise
- added C26, C27: 100n, Capacitor_SMD:C_0805_2012Metric, symbol Device:C
- added J17: Screw_Terminal_01x03, TerminalBlock:TerminalBlock_bornier-3_P5.08mm, symbol Connector:Screw_Terminal_01x03
- added R25: 1k, Resistor_SMD:R_1206_3216Metric, symbol Device:R
- added R26: 100, Resistor_SMD:R_1206_3216Metric, symbol Device:R
- added U6: MUX509ID, Package_SO:SOIC-16_3.9x9.9mm_P1.27mm, symbol Eli_v6Lib:MUX509ID
- R23: value DNP -> 100k
Connections:
- net +5VP: now also C26.1, U6.14 (VDD), U6.2 (EN)
- net -5V: now also C27.1, U6.3 (VSS)
- net GND: now also C26.2, C27.2, J17.1 (Pin_1), U6.15 (GND)
- net IMon+: now also R23.2, R24.2, R25.2, R26.2
- net IMon-: now also U6.8 (DrA)
- net IOut: now also R9.1
- net at R15.1, R2.1, U1.7: no longer R23.1
- net at BUF1.6 (Out), R10.1, R9.2: no longer R23.2, R24.2
- net Buf2Out: now reaches BUF2.6 (Out), J14.3 (Pin_3), J14.4 (Pin_4)
- net Buf2Out: now also U6.9 (DrB)
- net at R24.1: now also U6.12 (S2B), U6.5 (S2A)
- net InputSig: no longer names the net of J1.1 (In), R22.2
- new net: R25.1, U6.11 (S3B), U6.6 (S3A)
- new net: J17.3 (Pin_3), U6.1 (A0)
- new net: R26.1, U6.10 (S4B), U6.7 (S4A)
- new net: R23.1, U6.13 (S1B), U6.4 (S1A)
- new net: J17.2 (Pin_2), U6.16 (A1)
Other:
- note added: "OPA2810 is better suited 358 was used for standard footprint"
- note added: "Should be similar to shunt (R18 or 14) Does not need to be precision"
- note removed: "Buffer bypass Populate with 0 Ohm if buffer is not included Will limit ability to drive low impedance loads"
- note removed: "Input buffer and filter Selectable low-pass"
- note removed: "OPA2810 is better suited LMH6658MAX is a cheaper alternative Choose a fast opamp with R/R I/O 358 was used for standard footprint"
- note removed: "Should be similar to shunt (R18 or 14) for stability Does not need to be precision"
- moved on the sheet: BUF1, C1, C15, C16, C25, J1, J10, J12, J15, J16, J2, J3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
