File: Impedance_Analyzer_V4_KiCAD/6363_Connector.kicad_sch (KiCad schematic)
At the start: 26 parts, among them J1 5787362-7, K1 G6SK-2, Q1 IRLML0030, Q2 IRLML0030, Q20 IRLML0030, Q21 IRLML0030, Q22 IRLML0030, Q23 IRLML0030, Q3 IRLML0030, Q4 IRLML0030

Commit message: Initial Labview update
Parts:
- J1: footprint Eli_Lib:CONN68_5787362-7_TEC -> Eli_Lib:68DsubMaleTE_2-5174225-5
Changed lines of the file:
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@@
       (effects (font (size 1.524 1.524)))
     )
-    (property "Footprint" "Eli_Lib:CONN68_5787362-7_TEC" (id 2) (at 30.48 26.67 0)
+    (property "Footprint" "Eli_Lib:68DsubMaleTE_2-5174225-5" (id 2) (at 30.48 26.67 0)
       (effects (font (size 1.27 1.27) italic) hide)
     )
@@
       (effects (font (size 1.524 1.524)))
     )
-    (property "Footprint" "Eli_Lib:CONN68_5787362-7_TEC" (id 2) (at 63.5 110.49 0)
+    (property "Footprint" "Eli_Lib:68DsubMaleTE_2-5174225-5" (id 2) (at 63.5 110.49 0)
       (effects (font (size 1.27 1.27) italic) hide)
     )
