File: Impedance_Analyzer_V4_KiCAD/CurveTracer.kicad_sch (KiCad schematic)
At the start: 11 parts, among them J19 Conn_02x02_Counter_Clockwise, J20 Conn_Coaxial, J21 Conn_02x02_Counter_Clockwise, U1 AD8022, U7 INA129

Commit message: v4
Parts:
- U1: value AD8022 -> ADA4075-2; symbol Amplifier_Operational:LM358 -> Amplifier_Operational:ADA4075-2
Connections:
- net +5VP renamed +12V
- net -5V renamed -12V
Changed lines of the file:
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@@
     (pin "2")
   )
-  (symbol (lib_id "power:-5V") (at 190.5 114.3 0) (mirror x) (unit 1)
+  (symbol (lib_id "power:-12V") (at 190.5 114.3 0) (mirror x) (unit 1)
     (in_bom yes) (on_board yes)
-    (property "Reference" "#PWR0176" (id 0) (at 190.5 116.84 0)
+    (property "Reference" "#PWR0164" (id 0) (at 190.5 116.84 0)
       (effects (font (size 1.27 1.27)) hide)
     )
-    (property "Value" "-5V" (id 1) (at 190.881 118.6942 0))
+    (property "Value" "-12V" (id 1) (at 190.5 118.11 0))
     (property "Footprint" "" (id 2) (at 190.5 114.3 0)
       (effects (font (size 1.27 1.27)) hide)
@@
     (pin "2")
   )
-  (symbol (lib_id "Amplifier_Operational:LM358") (at 88.9 52.07 0) (unit 1)
+  (symbol (lib_id "Amplifier_Operational:ADA4075-2") (at 88.9 52.07 0) (unit 1)
     (in_bom yes) (on_board yes)
     (property "Reference" "U1" (id 0) (at 88.9 42.7482 0))
-    (property "Value" "AD8022" (id 1) (at 88.9 45.0596 0))
+    (property "Value" "ADA4075-2" (id 1) (at 88.9 57.15 0)
+      (effects (font (size 1.27 1.27)) (justify left))
+    )
     (property "Footprint" "Package_SO:SO-8_3.9x4.9mm_P1.27mm" (id 2) (at 88.9 52.07 0)
       (effects (font (size 1.27 1.27)) hide)
     )
-    (property "Datasheet" "http://www.ti.com/lit/ds/symlink/lm2904-n.pdf" (id 3) (at 88.9 52.07 0)
+    (property "Datasheet" "https://www.analog.com/static/imported-files/data_sheets/ADA4075-2.pdf" (id 3) (at 88.9 52.07 0)
       (effects (font (size 1.27 1.27)) hide)
     )
@@
     (pin "2")
     (pin "3")
+    (pin "5")
+    (pin "6")
+    (pin "7")
+    (pin "4")
+    (pin "8")
   )
   (symbol (lib_id "Device:R") (at 124.46 50.8 270) (unit 1)
@@
     (pin "2")
   )
-  (symbol (lib_id "power:+5VP") (at 190.5 88.9 0) (mirror y) (unit 1)
+  (symbol (lib_id "power:+12V") (at 190.5 88.9 0) (mirror y) (unit 1)
     (in_bom yes) (on_board yes)
-    (property "Reference" "#PWR0178" (id 0) (at 190.5 92.71 0)
+    (property "Reference" "#PWR0165" (id 0) (at 190.5 92.71 0)
       (effects (font (size 1.27 1.27)) hide)
     )
-    (property "Value" "+5VP" (id 1) (at 190.119 84.5058 0))
+    (property "Value" "+12V" (id 1) (at 190.5 85.344 0))
     (property "Footprint" "" (id 2) (at 190.5 88.9 0)
       (effects (font (size 1.27 1.27)) hide)
