File: Impedance_Analyzer_V4_KiCAD/Impedance_Analyzer_V4.kicad_pcb (KiCad board)
At the start: 4 copper layers, 98 x 101.6 mm, 114 parts, among them J1 5787362-7, J15 Conn_01x02_Male, J17 Conn_02x02_Counter_Clockwise, J18 Conn_01x02_Male, J19 Conn_02x02_Counter_Clockwise, J2 USB_B_Micro, J20 Conn_Coaxial, J21 Conn_02x02_Counter_Clockwise, J3 Conn_01x02_Male, J4 Conn_Coaxial, J5 Conn_Coaxial, J6 Conn_Coaxial, J7 Conn_Coaxial, J8 Conn_01x02_Male, K1 G6SK-2, K2 G6SK-2, Q1 IRLML0030, Q2 IRLML0030, Q20 IRLML0030, Q21 IRLML0030, Q22 IRLML0030, Q23 IRLML0030, Q3 IRLML0030, Q4 IRLML0030, U1 ADA4075-2, U2 ADA4075-2, U3 INA129, U4 INA129, U5 MC34063AD, U6 INA129, U7 INA129, U8 MC34063AD

Commit message: Initial Labview update
Parts:
- J1: footprint Eli_Lib:CONN68_5787362-7_TEC -> Eli_Lib:68DsubMaleTE_2-5174225-5; moved to F.Cu
- J2: footprint Connector_USB:USB_Micro-B_Wuerth_629105150521 -> Eli_Lib:AMPHENOL_10118194-0001LF
- TP1, TP2: footprint TestPoint:TestPoint_Plated_Hole_D3.0mm -> TestPoint:TestPoint_THTPad_2.0x2.0mm_Drill1.0mm
- moved J1 20.9 mm to (75.7, 85.0)
- moved J2 2.30 mm to (100.2, 141.0)
- moved C29 2.30 mm to (122.2, 137.0)
- moved C8 1.72 mm to (104.8, 117.0)
- moved L3 1.50 mm to (110.0, 119.5)
- moved K2 0.35 mm to (137.2, 130.0)
- turned L1 to 90 degrees
Connections:
- net Net-(C28-Pad1) renamed /Power_and_Inputs/+12VRaw
- net Net-(C4-Pad2) renamed /Power_and_Inputs/-12VRaw
Routing:
- net AI 3 (AI3+): track 0.00 -> 108.3 mm
- net +12V: track 219.7 -> 317.3 mm, vias 9 -> 13
- net P0.1: track 0.00 -> 96.3 mm, vias 0 -> 1
- net P0.2: track 0.00 -> 87.0 mm, vias 0 -> 1
- net AI1+: track 0.00 -> 83.9 mm
- net AI0+: track 0.00 -> 80.1 mm
- net P0.3: track 13.0 -> 89.7 mm
- net AI 2 (AI2+): track 0.00 -> 73.9 mm
- net P0.5: track 0.00 -> 69.8 mm, vias 0 -> 1
- net P0.0: track 22.4 -> 89.1 mm, vias 1 -> 2
- net P0.7: track 0.00 -> 64.7 mm, vias 0 -> 1
- net P0.4: track 0.00 -> 54.5 mm, vias 0 -> 1
- net P0.6: track 0.00 -> 54.1 mm, vias 0 -> 1
- net +5V-3: track 0.00 -> 52.2 mm
- net AO 0: track 0.00 -> 38.9 mm
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Other:
- board text added: "+12V"
- board text added: "-12V"
