File: Impedance_Analyzer_V4_KiCAD/Impedance_Analyzer_V4.kicad_sch (KiCad schematic)
At the start: 41 parts, among them J1 Conn_Coaxial_x2, J10 Conn_02x02_Counter_Clockwise, J11 Conn_Coaxial_x2, J12 Conn_02x02_Counter_Clockwise, J13 Conn_02x02_Counter_Clockwise, J14 Conn_02x02_Counter_Clockwise, J15 Conn_01x02_Male, J16 Conn_01x02_Male, J17 Conn_02x02_Counter_Clockwise, J18 Conn_01x02_Male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

Commit message: v4
Parts:
- removed J1, J11, J3: Conn_Coaxial_x2, Connector_Coaxial:BNC_Win_364A2x95_Horizontal, symbol Connector:Conn_Coaxial_x2
- removed J10, J12, J13, J14, J2: Conn_02x02_Counter_Clockwise, Connector_PinHeader_2.54mm:PinHeader_2x02_P2.54mm_Vertical, symbol Connector_Generic:Conn_02x02_Counter_Clockwise
- removed J16: Conn_01x02_Male, Connector_PinHeader_2.54mm:PinHeader_1x02_P2.54mm_Horizontal, symbol Connector:Conn_01x02_Male
- removed R11, R12, R25: 1k, Resistor_SMD:R_1206_3216Metric, symbol Device:R
- removed R13, R27, R5, R6: 0, Resistor_SMD:R_1206_3216Metric, symbol Device:R
- added D2, D3: 1N4148W, Diode_SMD:D_SOD-123, symbol Diode:1N4148W
- added K2: G6SK-2, Eli_Lib:RELAY_G6SK-2F DC3_OMR, symbol Relay:G6SK-2
- U1, U2: value AD8022 -> ADA4075-2; symbol Amplifier_Operational:LM358 -> Amplifier_Operational:ADA4075-2
Connections:
- net IMon+: now also K2.9; no longer R14.2, R18.2
- net IMon-: now also R14.1, R16.1, R18.1, U2.1
- net LPot1: now reaches J18.1 (Pin_1), J5.1 (In), U4.2 (-)
- net HPot1: now reaches J15.2 (Pin_2), J4.1 (In), U4.3 (+)
- net AI0+: now reaches U4.6
- net at U4.8 (Rg): now also R8.2
- net AI1+: now reaches U3.6
- net at U3.8 (Rg): now also R7.1
- net at R26.1: now also U6.8 (Rg)
- net AI 2 (AI2+): now reaches U6.6
- net +5VP renamed +12V
- net +12V: now also D2.1 (K), D3.1 (K), K2.1, K2.6
- net -5V renamed -12V
- net InputSig renamed AO 0
- new net: K2.10, R18.2
- new net: K2.8, R14.2
- new net R-: D2.2 (A), K2.7
- new net S-: D3.2 (A), K2.12
Other:
- added sheet DAQ Interface (6363_Connector.kicad_sch)
- moved on the sheet: R14, R18, R26, R7, R8
